File: PCB/Data-logger_v01-01/Data-logger_v01-01.brd (EAGLE design)
At the start: 162.2 x 105.4 mm, 33 parts, among them J1 6364372-1, Q4 LF33CV, U2 LPC1549JBD48, X1 22-23-2081, X2 22-23-2021, X3 87758-0416

Commit message: update components values
Parts:
- R2, R4: value 10k -> 1k1
- R3: value 10k -> 300R
Other:
- board text added: "nepropojena zem"
Changed lines of the file:
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@@
 <layers>
 <layer number="1" name="Top" color="4" fill="1" visible="yes" active="yes"/>
-<layer number="16" name="Bottom" color="1" fill="1" visible="no" active="yes"/>
+<layer number="16" name="Bottom" color="1" fill="1" visible="yes" active="yes"/>
 <layer number="17" name="Pads" color="2" fill="1" visible="yes" active="yes"/>
 <layer number="18" name="Vias" color="2" fill="1" visible="yes" active="yes"/>
@@
 <layer number="48" name="Document" color="7" fill="1" visible="no" active="yes"/>
 <layer number="49" name="Reference" color="7" fill="1" visible="no" active="yes"/>
-<layer number="51" name="tDocu" color="7" fill="1" visible="no" active="yes"/>
-<layer number="52" name="bDocu" color="7" fill="1" visible="no" active="yes"/>
+<layer number="51" name="tDocu" color="7" fill="1" visible="yes" active="yes"/>
+<layer number="52" name="bDocu" color="7" fill="1" visible="yes" active="yes"/>
 <layer number="88" name="SimResults" color="9" fill="1" visible="no" active="no"/>
 <layer number="89" name="SimProbes" color="9" fill="1" visible="no" active="no"/>
@@
 FEKT 2025
 BP V01-01</text>
+<text x="44.45" y="20.32" size="1.778" layer="51">nepropojena zem</text>
 </plain>
 <attributes>
@@
 <attribute name="VALUE" x="43.18" y="61.945" size="1.27" layer="27" rot="R270"/>
 </element>
-<element name="R2" library="rcl" library_urn="urn:adsk.eagle:library:334" package="R1206W" package3d_urn="urn:adsk.eagle:package:23539/2" value="10k" x="43.18" y="53.34" smashed="yes" rot="R270">
+<element name="R2" library="rcl" library_urn="urn:adsk.eagle:library:334" package="R1206W" package3d_urn="urn:adsk.eagle:package:23539/2" value="1k1" x="43.18" y="53.34" smashed="yes" rot="R270">
 <attribute name="NAME" x="44.45" y="55.245" size="1.27" layer="25" rot="R270"/>
 <attribute name="POPULARITY" value="3" x="43.18" y="53.34" size="1.778" layer="27" rot="R270" display="off"/>
@@
 <attribute name="VALUE" x="40.64" y="55.245" size="1.27" layer="27" rot="R270"/>
 </element>
-<element name="R3" library="rcl" library_urn="urn:adsk.eagle:library:334" package="R1206W" package3d_urn="urn:adsk.eagle:package:23539/2" value="10k" x="47.625" y="53.975" smashed="yes">
+<element name="R3" library="rcl" library_urn="urn:adsk.eagle:library:334" package="R1206W" package3d_urn="urn:adsk.eagle:package:23539/2" value="300R" x="47.625" y="53.975" smashed="yes">
 <attribute name="NAME" x="45.72" y="55.245" size="1.27" layer="25"/>
 <attribute name="POPULARITY" value="3" x="47.625" y="53.975" size="1.778" layer="27" display="off"/>
@@
 <attribute name="VALUE" x="45.72" y="51.435" size="1.27" layer="27"/>
 </element>
-<element name="R4" library="rcl" library_urn="urn:adsk.eagle:library:334" package="R1206W" package3d_urn="urn:adsk.eagle:package:23539/2" value="10k" x="39.37" y="53.34" smashed="yes" rot="R270">
+<element name="R4" library="rcl" library_urn="urn:adsk.eagle:library:334" package="R1206W" package3d_urn="urn:adsk.eagle:package:23539/2" value="1k1" x="39.37" y="53.34" smashed="yes" rot="R270">
 <attribute name="NAME" x="40.64" y="55.245" size="1.27" layer="25" rot="R270"/>
 <attribute name="POPULARITY" value="3" x="39.37" y="53.34" size="1.778" layer="27" rot="R270" display="off"/>
